Commit message: Magnetometer added to some files (Hector_gazebo not added)

File: eufs_racecar/robots/ads-dv/robot.urdf.xacro (robot description, xacro)
@@ -55,3 +55,6 @@
         <origin xyz="0.334 0.0 0.295" rpy="0 ${10.15*M_PI/180.0} 0"/>
     </xacro:sensor_imu>
+    <xacro:sensor_magnetometer parent="base_footprint" prefix="sbg">
+        <origin xyz="0.0 0.0 0.0" rpy="0 0 0"/>
+    </xacro:sensor_magnetometer>
 </robot>

File: eufs_racecar/robots/eufs/robot.urdf.xacro (robot description, xacro)
@@ -55,3 +55,6 @@
         <origin xyz="-0.08 0.0 0.76" rpy="0 0 0"/>
     </xacro:sensor_imu>
+    <xacro:sensor_magnetometer parent="base_footprint" prefix="sbg">
+        <origin xyz="0.0 0.0 0.0" rpy="0 0 0"/>
+    </xacro:sensor_magnetometer>
 </robot>

File: eufs_sensors/urdf/all_sensors.urdf.xacro (robot description, xacro)
@@ -6,4 +6,6 @@
   <!-- Velodyne VLP-16R -->
   <xacro:include filename="$(find eufs_sensors)/urdf/VLP-16R.urdf.xacro"/>
+  <!-- Magnetometer-->
+  <xacro:include filename="$(find eufs_sensors)/urdf/magnetometer.urdf.xacro"/>
   <!--IMU -->
   <xacro:include filename="$(find eufs_sensors)/urdf/imu.urdf.xacro"/>
